File: pcb/tartan.kicad_pcb (KiCad board)
At the start: 2 copper layers, 285 x 117 mm, 171 parts, among them J1 AVR_ISP_6, J2 USB_OTG, SW1 SW_Push, SW10 SW_Push, SW11 SW_Push, SW12 SW_Push, SW13 SW_Push, SW14 SW_Push, SW15 SW_Push, SW16 SW_Push, SW17 SW_Push, SW18 SW_Push, SW19 SW_Push, SW2 SW_Push, SW20 SW_Push, SW21 SW_Push, SW22 SW_Push, SW23 SW_Push, SW24 SW_Push, SW25 SW_Push, SW26 SW_Push, SW27 SW_Push, SW28 SW_Push, SW29 SW_Push, SW3 SW_Push, SW30 SW_Push, SW31 SW_Push, SW32 SW_Push, SW33 SW_Push, SW34 SW_Push, SW35 SW_Push, SW36 SW_Push, SW37 SW_Push, SW38 SW_Push, SW39 SW_Push, SW4 SW_Push, SW40 SW_Push, SW41 SW_Push, SW42 SW_Push, SW43 SW_Push, SW44 SW_Push, SW45 SW_Push, SW46 SW_Push, SW47 SW_Push, SW48 SW_Push, SW49 SW_Push, SW5 SW_Push, SW50 SW_Push, SW51 SW_Push, SW52 SW_Push, SW53 SW_Push, SW54 SW_Push, SW55 SW_Push, SW56 SW_Push, SW57 SW_Push, SW58 SW_Push, SW59 SW_Push, SW6 SW_Push, SW60 SW_Push, SW61 SW_Push, SW62 SW_Push, SW63 SW_Push, SW64 SW_Push, SW65 SW_Push, SW66 SW_Push, SW67 SW_Push, SW68 SW_Push, SW69 SW_Push, SW7 SW_Push, SW70 RESET, SW71 BOOT, SW8 SW_Push, SW9 SW_Push, U1 ATMEGA328-PU, Y1 16MHz

Commit message: Add files via upload
Parts:
- moved D11 157.6 mm to (42.6, 41.5)
- moved D62 35.6 mm to (108.7, 41.5)
- moved D56 33.1 mm to (195.2, 41.4)
- moved D61 30.5 mm to (96.0, 41.5)
- moved D24 30.4 mm to (144.4, 41.4)
- moved D29 25.5 mm to (197.7, 41.4)
- moved D53 25.5 mm to (159.6, 41.4)
- moved D25 25.4 mm to (151.9, 41.5)
- moved D23 22.9 mm to (136.6, 41.5)
- moved D63 22.9 mm to (174.8, 41.4)
- moved D51 22.9 mm to (139.2, 41.5)
- moved D55 20.4 mm to (177.4, 41.4)
- moved D54 20.4 mm to (167.2, 41.4)
- moved D49 20.3 mm to (121.4, 41.5)
- moved D50 20.3 mm to (131.5, 41.5)
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Routing:
- net Net-(D11-Pad2): track 44.9 -> 305.3 mm
- net /COL10: track 160.5 -> 327.7 mm, vias 2 -> 0
- net /COL9: track 167.0 -> 294.0 mm, vias 1 -> 0
- net /COL11: track 129.0 -> 204.9 mm
- net Net-(D61-Pad2): track 155.0 -> 210.3 mm
- net /ROW0: track 213.3 -> 267.6 mm
- net /ROW1: track 210.0 -> 263.4 mm
- net Net-(D62-Pad2): track 167.5 -> 220.3 mm
- net Net-(D60-Pad2): track 121.8 -> 161.7 mm
- net Net-(D58-Pad2): track 100.4 -> 134.0 mm
- net /COL4: track 274.6 -> 304.3 mm, vias 1 -> 0
- net Net-(D29-Pad2): track 171.9 -> 144.0 mm
- net Net-(D24-Pad2): track 44.4 -> 71.2 mm
- net Net-(D64-Pad2): track 201.9 -> 226.0 mm
- net Net-(D13-Pad2): track 87.8 -> 111.5 mm
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